File: pcb/pinky/skean.kicad_sch (KiCad schematic)
At the start: 77 parts, among them J2 SWD, J3 USB-C Conn, J4 Conn_01x02_Female, K10 KEYSW, K11 KEYSW, K12 KEYSW, K13 KEYSW, K14 KEYSW, K15 KEYSW, K16 KEYSW, K17 KEYSW, K18 KEYSW, K19 KEYSW, K2 KEYSW, K20 KEYSW, K21 KEYSW, K22 KEYSW, K3 KEYSW, K4 KEYSW, K5 KEYSW, K6 KEYSW, K7 KEYSW, K8 KEYSW, K9 KEYSW, Q2 AO3407, SW1 SW_SPDT, U1 E73-2G4M08S1E, U2 XC6220B331MR-G, U3 TP4054, U4 USBLC6-2SC6, X1 32.768kHz

Commit message: близко
Parts:
- added K1: KEYSW, kbd:MX-Alps-1U-REV, symbol Keyboard_Components:KEYSW
Connections:
- net COL0: now also K1.2 (B)
- net at D1.2 (A): now also K1.1 (A)
Changed lines of the file:
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@@
+    (pin "2")
+  )
+  (symbol (lib_id "Keyboard_Components:KEYSW") (at 62.23 97.79 0) (unit 1)
+    (in_bom yes) (on_board yes)
+    (property "Reference" "K1" (id 0) (at 62.23 91.44 0))
+    (property "Value" "KEYSW" (id 1) (at 62.23 93.98 0))
+    (property "Footprint" "kbd:MX-Alps-1U-REV" (id 2) (at 62.23 92.71 0)
+      (effects (font (size 1.27 1.27)) hide)
+    )
+    (property "Datasheet" "~" (id 3) (at 62.23 97.79 0)
+      (effects (font (size 1.27 1.27)) hide)
+    )
+    (pin "1")
     (pin "2")
   )
@@
       (reference "J4") (unit 1) (value "Conn_01x02_Female") (footprint "kbd:Battery_TH")
     )
+    (path "/bc531e3f-fe79-4957-a649-1376b3436c93"
+      (reference "K1") (unit 1) (value "KEYSW") (footprint "kbd:MX-Alps-1U-REV")
+    )
     (path "/ca0b9cf6-1ae9-4c0a-9012-8b74ea50e4d2"
